File: tests/reference-outputs/project-with-kicad-lib/loclib/project-with-kicad-lib.kicad_sch (KiCad schematic)
At the start: 6 parts, among them U1 ADS1115IDGS

Commit message: [#63388] tests: Add tests for loclib
Parts:
- C1: footprint Capacitor_SMD:C_0402_1005Metric_Pad0.74x0.62mm_HandSolder -> project-with-kicad-lib-footprints:C_0402_1005Metric_Pad0.74x0.62mm_HandSolder; symbol Device:C_Small -> project-with-kicad-lib:C_Small
- D1: footprint LED_THT:LED_D5.0mm -> project-with-kicad-lib-footprints:LED_D5.0mm; symbol Device:LED -> project-with-kicad-lib:LED
- R1, R2, R3: footprint Resistor_SMD:R_0402_1005Metric_Pad0.72x0.64mm_HandSolder -> project-with-kicad-lib-footprints:R_0402_1005Metric_Pad0.72x0.64mm_HandSolder; symbol Device:R_Small -> project-with-kicad-lib:R_Small
- U1: footprint Package_SO:TSSOP-10_3x3mm_P0.5mm -> project-with-kicad-lib-footprints:TSSOP-10_3x3mm_P0.5mm; symbol Analog_ADC:ADS1115IDGS -> project-with-kicad-lib:ADS1115IDGS
Changed lines of the file:
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@@
     (stroke (width 0) (type default))
   )
-  (symbol (lib_id "power:GND") (at 121.92 85.09 0) (unit 1)
+  (symbol (lib_id "project-with-kicad-lib:GND") (at 121.92 85.09 0) (unit 1)
     (in_bom yes) (on_board yes) (dnp no) (fields_autoplaced)
     (property "Reference" "#PWR03" (at 130.81 87.63 0)
@@
     )
   )
-  (symbol (lib_id "power:+3.3V") (at 162.56 74.93 0) (unit 1)
+  (symbol (lib_id "project-with-kicad-lib:+3.3V") (at 162.56 74.93 0) (unit 1)
     (in_bom yes) (on_board yes) (dnp no) (fields_autoplaced)
     (property "Reference" "#PWR04" (at 162.56 78.74 0)
@@
     )
   )
-  (symbol (lib_id "power:GND") (at 107.95 106.68 0) (unit 1)
+  (symbol (lib_id "project-with-kicad-lib:GND") (at 107.95 106.68 0) (unit 1)
     (in_bom yes) (on_board yes) (dnp no) (fields_autoplaced)
     (property "Reference" "#PWR06" (at 116.84 109.22 0)
@@
     )
   )
-  (symbol (lib_id "Device:R_Small") (at 166.37 86.36 0) (unit 1)
+  (symbol (lib_id "project-with-kicad-lib:R_Small") (at 166.37 86.36 0) (unit 1)
     (in_bom yes) (on_board yes) (dnp no)
     (property "Reference" "R2" (at 167.64 85.09 0)
@@
       (effects (font (size 1.27 1.27)) (justify left))
     )
-    (property "Footprint" "Resistor_SMD:R_0402_1005Metric_Pad0.72x0.64mm_HandSolder" (at 166.37 86.36 0)
+    (property "Footprint" "project-with-kicad-lib-footprints:R_0402_1005Metric_Pad0.72x0.64mm_HandSolder" (at 166.37 86.36 0)
       (effects (font (size 1.27 1.27)) hide)
     )
@@
     )
   )
-  (symbol (lib_id "power:+3.3V") (at 139.7 74.93 0) (unit 1)
+  (symbol (lib_id "project-with-kicad-lib:+3.3V") (at 139.7 74.93 0) (unit 1)
     (in_bom yes) (on_board yes) (dnp no) (fields_autoplaced)
     (property "Reference" "#PWR02" (at 139.7 78.74 0)
@@
     )
   )
-  (symbol (lib_id "Device:LED") (at 107.95 95.25 90) (unit 1)
+  (symbol (lib_id "project-with-kicad-lib:LED") (at 107.95 95.25 90) (unit 1)
     (in_bom yes) (on_board yes) (dnp no) (fields_autoplaced)
     (property "Reference" "D1" (at 111.76 95.5675 90)
@@
       (effects (font (size 1.27 1.27)) (justify right))
     )
-    (property "Footprint" "LED_THT:LED_D5.0mm" (at 107.95 95.25 0)
+    (property "Footprint" "project-with-kicad-lib-footprints:LED_D5.0mm" (at 107.95 95.25 0)
       (effects (font (size 1.27 1.27)) hide)
     )
@@
     )
   )
-  (symbol (lib_id "Analog_ADC:ADS1115IDGS") (at 139.7 92.71 0) (unit 1)
+  (symbol (lib_id "project-with-kicad-lib:ADS1115IDGS") (at 139.7 92.71 0) (unit 1)
     (in_bom yes) (on_board yes) (dnp no) (fields_autoplaced)
     (property "Reference" "U1" (at 141.8941 77.47 0)
@@
       (effects (font (size 1.27 1.27)) (justify left))
     )
-    (property "Footprint" "Package_SO:TSSOP-10_3x3mm_P0.5mm" (at 139.7 105.41 0)
+    (property "Footprint" "project-with-kicad-lib-footprints:TSSOP-10_3x3mm_P0.5mm" (at 139.7 105.41 0)
       (effects (font (size 1.27 1.27)) hide)
     )
@@
     )
   )
-  (symbol (lib_id "power:+3.3V") (at 107.95 74.93 0) (unit 1)
+  (symbol (lib_id "project-with-kicad-lib:+3.3V") (at 107.95 74.93 0) (unit 1)
     (in_bom yes) (on_board yes) (dnp no) (fields_autoplaced)
     (property "Reference" "#PWR05" (at 107.95 78.74 0)
@@
     )
   )
-  (symbol (lib_id "power:GND") (at 139.7 106.68 0) (unit 1)
+  (symbol (lib_id "project-with-kicad-lib:GND") (at 139.7 106.68 0) (unit 1)
     (in_bom yes) (on_board yes) (dnp no) (fields_autoplaced)
     (property "Reference" "#PWR01" (at 148.59 109.22 0)
@@
     )
   )
-  (symbol (lib_id "Device:R_Small") (at 107.95 83.82 0) (unit 1)
+  (symbol (lib_id "project-with-kicad-lib:R_Small") (at 107.95 83.82 0) (unit 1)
     (in_bom yes) (on_board yes) (dnp no)
     (property "Reference" "R3" (at 109.22 82.55 0)
@@
       (effects (font (size 1.27 1.27)) (justify left))
     )
-    (property "Footprint" "Resistor_SMD:R_0402_1005Metric_Pad0.72x0.64mm_HandSolder" (at 107.95 83.82 0)
+    (property "Footprint" "project-with-kicad-lib-footprints:R_0402_1005Metric_Pad0.72x0.64mm_HandSolder" (at 107.95 83.82 0)
       (effects (font (size 1.27 1.27)) hide)
     )
@@
     )
   )
-  (symbol (lib_id "Device:C_Small") (at 121.92 81.28 0) (unit 1)
+  (symbol (lib_id "project-with-kicad-lib:C_Small") (at 121.92 81.28 0) (unit 1)
     (in_bom yes) (on_board yes) (dnp no) (fields_autoplaced)
     (property "Reference" "C1" (at 124.46 80.0163 0)
@@
       (effects (font (size 1.27 1.27)) (justify left))
     )
-    (property "Footprint" "Capacitor_SMD:C_0402_1005Metric_Pad0.74x0.62mm_HandSolder" (at 121.92 81.28 0)
+    (property "Footprint" "project-with-kicad-lib-footprints:C_0402_1005Metric_Pad0.74x0.62mm_HandSolder" (at 121.92 81.28 0)
       (effects (font (size 1.27 1.27)) hide)
     )
@@
     )
   )
-  (symbol (lib_id "Device:R_Small") (at 158.75 86.36 0) (unit 1)
+  (symbol (lib_id "project-with-kicad-lib:R_Small") (at 158.75 86.36 0) (unit 1)
     (in_bom yes) (on_board yes) (dnp no)
     (property "Reference" "R1" (at 160.02 85.09 0)
@@
       (effects (font (size 1.27 1.27)) (justify left))
     )
-    (property "Footprint" "Resistor_SMD:R_0402_1005Metric_Pad0.72x0.64mm_HandSolder" (at 158.75 86.36 0)
-      (effects (font (size 1.27 1.27)) hide)
-    )
+    (property "Footprint" "project-with-kicad-lib-footprints:R_0402_1005Metric_Pad0.72x0.64mm_HandSolder" (at 158.75 86.36 0)
+      (effects (font (size 1.27 1.27)) hide)
+    )
