File: tests/reference-outputs/loclib/connectors.kicad_sch (KiCad schematic)
At the start: 5 parts, among them J1 HDMI_A, J2 Conn_01x02_Pin, J4 Conn_01x35_Pin

Commit message: [#70870] Update test design rebase
Parts:
- added D3: PESD3V3L4UG, test_project-footprints:SOT-353_SC-70-5, symbol test_project:PESD3V3L4UG
Connections:
- net GND: now also D3.2 (A)
- net hdmi_in.CEC: now also D3.1 (K1)
- net hdmi_in.HPD: now also D3.5 (K4)
- net hdmi_in.SCL: now also D3.3 (K2)
- net hdmi_in.SDA: now also D3.4 (K3)

Commit message: [#75441] Kicad9
Parts:
- J1: Component Class (none) -> CONNECTOR
