File: tests/reference-outputs/loclib/power.kicad_sch (KiCad schematic)
At the start: 19 parts, among them J3 Barrel_Jack_MountingPin, U3 LM3880, U4 AP2112K-1.8, U6 RT9742AGJ5F

Commit message: [#70870] Update test design rebase
Parts:
- added R12, R8: 220, test_project-footprints:R_0402_1005Metric, symbol test_project:R
Connections:
- no-connect marks 1 -> 5
Changed lines of the file:
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@@
 (kicad_sch (version 20231120) (generator "eeschema") (generator_version "8.0")
   (paper "A4")
+  (junction (at 201.93 83.82) (diameter 0) (color 0 0 0 0)
+  )
   (junction (at 106.68 104.14) (diameter 0) (color 0 0 0 0)
   )
@@
   (junction (at 166.37 85.09) (diameter 0) (color 0 0 0 0)
   )
+  (no_connect (at 273.05 139.7))
+  (no_connect (at 265.43 147.32))
   (no_connect (at 127 116.84))
+  (no_connect (at 265.43 139.7))
+  (no_connect (at 273.05 147.32))
   (wire (pts (xy 102.87 104.14) (xy 106.68 104.14))
     (stroke (width 0) (type default))
@@
     (stroke (width 0) (type default))
   )
-  (wire (pts (xy 201.93 95.25) (xy 201.93 83.82))
-    (stroke (width 0) (type default))
-  )
   (wire (pts (xy 166.37 85.09) (xy 166.37 83.82))
     (stroke (width 0) (type default))
@@
     (stroke (width 0) (type default))
   )
+  (wire (pts (xy 201.93 83.82) (xy 207.01 83.82))
+    (stroke (width 0) (type default))
+  )
   (wire (pts (xy 232.41 97.79) (xy 232.41 100.33))
     (stroke (width 0) (type default))
@@
     (stroke (width 0) (type default))
   )
+  (wire (pts (xy 201.93 83.82) (xy 201.93 95.25))
+    (stroke (width 0) (type default))
+  )
   (wire (pts (xy 74.93 102.87) (xy 74.93 110.49))
     (stroke (width 0) (type default))
@@
   (wire (pts (xy 187.96 100.33) (xy 187.96 85.09))
     (stroke (width 0) (type default))
+  )
+  (netclass_flag "" (length 2.54) (shape round) (at 207.01 83.82 0) (fields_autoplaced yes)
+    (effects (font (size 1.27 1.27)) (justify left bottom))
+    (property "Netclass" "power" (at 207.7085 81.28 0)
+      (effects (font (size 1.27 1.27) (italic yes)) (justify left))
+    )
   )
   (symbol (lib_id "test_project:+1V8") (at 201.93 121.92 0) (unit 1) (exclude_from_sim no)
@@
         (path "/59f522e0-0cf7-48a6-bc09-47b340553d24/9fb9e3b9-702c-4bf6-8780-47a0645875b6"
           (reference "#PWR012") (unit 1)
+        )
+      )
+    )
+  )
+  (symbol (lib_id "test_project:R") (at 273.05 143.51 0) (unit 1) (exclude_from_sim no)
+    (in_bom yes) (on_board yes) (dnp no) (fields_autoplaced yes)
+    (property "Reference" "R12" (at 275.59 142.2399 0)
+      (effects (font (size 1.27 1.27)) (justify left))
+    )
+    (property "Value" "220" (at 275.59 144.7799 0)
+      (effects (font (size 1.27 1.27)) (justify left))
+    )
+    (property "Footprint" "test_project-footprints:R_0402_1005Metric" (at 271.272 143.51 90)
+      (effects (font (size 1.27 1.27))( hide yes ))
+    )
+    (property "Datasheet" "~" (at 273.05 143.51 0)
+      (effects (font (size 1.27 1.27))( hide yes ))
+    )
+    (property "Description" "Resistor" (at 273.05 143.51 0)
+      (effects (font (size 1.27 1.27))( hide yes ))
+    )
+  (pin  "1")
+  (pin  "2")
+    (instances
+      (project "test_project"
+        (path "/59f522e0-0cf7-48a6-bc09-47b340553d24/9fb9e3b9-702c-4bf6-8780-47a0645875b6"
+          (reference "R12") (unit 1)
         )
       )
@@
         )
       )
+    )
+  )
+  (symbol (lib_id "test_project:R") (at 265.43 143.51 0) (unit 1) (exclude_from_sim no)
+    (in_bom yes) (on_board yes) (dnp no) (fields_autoplaced yes)
+    (property "Reference" "R8" (at 267.97 142.2399 0)
+      (effects (font (size 1.27 1.27)) (justify left))
+    )
+    (property "Value" "220" (at 267.97 144.7799 0)
+      (effects (font (size 1.27 1.27)) (justify left))
+    )
+    (property "Footprint" "test_project-footprints:R_0402_1005Metric" (at 263.652 143.51 90)
+      (effects (font (size 1.27 1.27))( hide yes ))
+    )
+    (property "Datasheet" "~" (at 265.43 143.51 0)
+      (effects (font (size 1.27 1.27))( hide yes ))
+    )
+    (property "Description" "Resistor" (at 265.43 143.51 0)
+      (effects (font (size 1.27 1.27))( hide yes ))
+    )
+  (pin  "1")
+  (pin  "2")
+    (instances
+      (project "test_project"
+        (path "/59f522e0-0cf7-48a6-bc09-47b340553d24/9fb9e3b9-702c-4bf6-8780-47a0645875b6"
+          (reference "R8") (unit 1)
+        )
+      )

Commit message: [#75441] Kicad9
Parts:
- R8: TODO (none) -> ${ERC_ERROR TODO}Manual ERC error (sym field)
Other:
- note added: "${ERC_WARNING "TODO Fill Table"} Manual ERC warning"
