File: tests/reference-outputs/loclib/test_project.kicad_sch (KiCad schematic)
At the start: 4 parts

Commit message: [#70870] Update test design rebase
Parts:
- removed H4: MountingHole_Pad, test_project-footprints:MountingHole_2.2mm_M2_DIN965_Pad, symbol test_project:MountingHole_Pad
Other:
- note added: "Arc > 180 deg"
- note added: "Non default font text"
- note added: "PNG image"
Changed lines of the file:
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@@
   (junction (at 365.76 226.06) (diameter 0) (color 0 0 0 0)
   )
-  (junction (at 365.76 236.22) (diameter 0) (color 0 0 0 0)
-  )
   (polyline (pts (xy 198.2523 106.1244) (xy 207.1502 106.1244))
     (stroke (width 0) (type solid))
@@
     (stroke (width 0) (type default))
   )
-  (polyline (pts (xy 251.1531 158.414) (xy 250.9414 135.5751))
+  (polyline (pts (xy 250.9368 157.9439) (xy 250.9414 135.5751))
     (stroke (width 0) (type solid))
   )
@@
     (stroke (width 0) (type default))
   )
-  (wire (pts (xy 365.76 231.14) (xy 365.76 236.22))
-    (stroke (width 0) (type default))
-  )
-  (wire (pts (xy 365.76 236.22) (xy 365.76 240.03))
+  (wire (pts (xy 365.76 231.14) (xy 365.76 240.03))
     (stroke (width 0) (type default))
   )
@@
     (stroke (width 0) (type solid))
   )
-  (polyline (pts (xy 265.6258 134.0326) (xy 265.7237 158.2976))
+  (polyline (pts (xy 265.6258 134.0326) (xy 265.6407 157.9838))
     (stroke (width 0) (type solid))
   )
@@
   (polyline (pts (xy 208.5393 95.5463) (xy 206.7031 96.5015) (xy 207.1502 95.5675) (xy 206.674 94.6494) (xy 208.5393 95.5463))
     (stroke (width 0) (type solid))
-    (fill (type outline))
+    (fill (type color) (color 0 0 0 0))
   )
   (polyline (pts (xy 237.6435 120.5865) (xy 235.7914 121.5125) (xy 236.2544 120.5865) (xy 235.7914 119.6605) (xy 237.6435 120.5865))
     (stroke (width 0) (type solid))
-    (fill (type outline))
+    (fill (type color) (color 0 0 0 0))
   )
   (polyline (pts (xy 208.5393 106.1244) (xy 206.6872 107.0504) (xy 207.1502 106.1244) (xy 206.6872 105.1983) (xy 208.5393 106.1244))
     (stroke (width 0) (type solid))
-    (fill (type outline))
+    (fill (type color) (color 0 0 0 0))
   )
   (polyline (pts (xy 203.544 141.8431) (xy 171.794 141.8431) (xy 171.794 125.9681) (xy 203.544 125.9681) (xy 203.544 141.8431))
@@
   (polyline (pts (xy 174.1435 102.1556) (xy 172.2914 103.0817) (xy 172.7544 102.1556) (xy 172.2914 101.2296) (xy 174.1435 102.1556))
     (stroke (width 0) (type solid))
-    (fill (type outline))
-  )
-  (polyline (pts (xy 251.1663 159.803) (xy 250.2217 157.9589) (xy 251.1531 158.414) (xy 252.0738 157.943) (xy 251.1663 159.803))
-    (stroke (width 0) (type solid))
-    (fill (type outline))
+    (fill (type color) (color 0 0 0 0))
+  )
+  (polyline (pts (xy 250.9966 159.6345) (xy 250.052 157.7904) (xy 250.9834 158.2455) (xy 251.9041 157.7745) (xy 250.9966 159.6345))
+    (stroke (width 0) (type solid))
+    (fill (type color) (color 0 0 0 0))
   )
   (polyline (pts (xy 158.5648 110.0931) (xy 134.7523 110.0931) (xy 134.7523 94.2181) (xy 158.5648 94.2181) (xy 158.5648 110.0931))
@@
   (polyline (pts (xy 237.6435 129.9369) (xy 235.7914 130.8629) (xy 236.2544 129.9369) (xy 235.7914 129.0108) (xy 237.6435 129.9369))
     (stroke (width 0) (type solid))
-    (fill (type outline))
+    (fill (type color) (color 0 0 0 0))
   )
   (polyline (pts (xy 269.6898 133.9056) (xy 237.9398 133.9056) (xy 237.9398 118.0306) (xy 269.6898 118.0306) (xy 269.6898 133.9056))
@@
   (polyline (pts (xy 287.9143 125.9681) (xy 286.0622 126.8942) (xy 286.5252 125.9681) (xy 286.0622 125.0421) (xy 287.9143 125.9681))
     (stroke (width 0) (type solid))
-    (fill (type outline))
+    (fill (type color) (color 0 0 0 0))
   )
   (polyline (pts (xy 198.2523 110.0931) (xy 174.4398 110.0931) (xy 174.4398 94.2181) (xy 198.2523 94.2181) (xy 198.2523 110.0931))
@@
   (polyline (pts (xy 251.8727 136.0302) (xy 250.9414 135.5751) (xy 250.0207 136.0461) (xy 250.9282 134.1861) (xy 251.8727 136.0302))
     (stroke (width 0) (type solid))
-    (fill (type outline))
+    (fill (type color) (color 0 0 0 0))
   )
   (polyline (pts (xy 240.5856 99.5098) (xy 208.8356 99.5098) (xy 208.8356 91.5723) (xy 240.5856 91.5723) (xy 240.5856 99.5098))
@@
   (polyline (pts (xy 261.7523 117.4697) (xy 260.8262 115.6176) (xy 261.7523 116.0806) (xy 262.6783 115.6176) (xy 261.7523 117.4697))
     (stroke (width 0) (type solid))
-    (fill (type outline))
-  )
-  (polyline (pts (xy 265.7316 159.6866) (xy 264.7976 157.8398) (xy 265.7237 158.2976) (xy 266.6497 157.8319) (xy 265.7316 159.6866))
-    (stroke (width 0) (type solid))
-    (fill (type outline))
+    (fill (type color) (color 0 0 0 0))
+  )
+  (polyline (pts (xy 265.6633 159.6377) (xy 264.7293 157.7909) (xy 265.6554 158.2487) (xy 266.5814 157.783) (xy 265.6633 159.6377))
+    (stroke (width 0) (type solid))
+    (fill (type color) (color 0 0 0 0))
   )
   (polyline (pts (xy 312.0231 133.9056) (xy 288.2106 133.9056) (xy 288.2106 118.0306) (xy 312.0231 118.0306) (xy 312.0231 133.9056))
@@
   (polyline (pts (xy 245.8773 117.2051) (xy 244.9512 115.353) (xy 245.8773 115.8161) (xy 246.8033 115.353) (xy 245.8773 117.2051))
     (stroke (width 0) (type solid))
-    (fill (type outline))
+    (fill (type color) (color 0 0 0 0))
+  )
+  (arc (start 49.53 219.71) (mid 30.6664 215.265) (end 49.53 210.82)
+    (stroke (width 0) (type default))
+    (fill (type none))
+  )
+  (image (at 41.91 186.69)
+    (data
+      "iVBORw0KGgoAAAANSUhEUgAAASwAAABkCAIAAACzY5qXAAABhWlDQ1BJQ0MgcHJvZmlsZQAAKJF9"
+      "kT1Iw0AcxV9TpVIrDmYQcchQnayDiggutQpFqBBqhVYdzEe/oElDkuLiKLgWHPxYrDq4OOvq4CoI"
+      "gh8gzg5Oii5S4v+SQosYD4778e7e4+4dwDUqimZ1xQFNt810MiFkc6tC6BW94BHGOGYlxTLmRDEF"
+      "3/F1jwBb72Isy//cn6NPzVsKEBCI44ph2sQbxNObtsF4n5hXSpJKfE48ZtIFiR+ZLnv8xrjoMscy"
+      "eTOTnifmiYViB8sdrJRMjXiKOKpqOuVzWY9VxluMtUpNad2TvTCS11eWmU5zGEksYgkiBMiooYwK"
+      "bMRo1UmxkKb9hI9/yPWL5JLJVYZCjgVUoUFy/WB/8LtbqzA54SVFEkD3i+N8jAChXaBZd5zvY8dp"
+      "ngDBZ+BKb/urDWDmk/R6W4seAf3bwMV1W5P3gMsdYPDJkEzJlYI0uUIBeD+jb8oBA7dAeM3rrbWP"
+      "0wcgQ12lboCDQ2C0SNnrPu/u6ezt3zOt/n4AClhy4x7yWMEAAAAJcEhZcwAALiMAAC4jAXilP3YA"
+      "AADwSURBVHja7dNBDQAgEAPBO6yBbNAGFvolmZHQdPsWkbNrTTPE2rNSwwQgQhAhIEIQISBCECEg"
+      "QhAhIEIQISBCECEgQhAhIEIQISBCECEgQhAhIEIQISBCECEgQhAhIEIQISBCECEgQhAhIEIQISBC"
+      "ECEgQhAhIEIQISBCECEgQhAhIEIQISBCECEgQhAhIEIQISBCECEgQhAhIEIQISBCECEgQhAhIEIQ"
+      "IYgQECGIEBAhiBAQIYgQECGIEBAhiBAQIYgQECGIEBAhiBAQIYgQECGIEBAhiBAQIYgQECGIEBAh"
+      "iBAQIYgQECGIEBAh/OwB8voExzrxYwwAAAAASUVORK5CYII="
+    )
   )
   (text "Control"  (exclude_from_sim no)(at 252.984 146.558 90)
     (effects (font (size 1.27 1.27)))
   )
+  (text "Arc > 180 deg"  (exclude_from_sim no)(at 40.894 215.646 0)
+    (effects (font (size 1.27 1.27)))
+  )
+  (text "PNG image"  (exclude_from_sim no)(at 41.91 180.848 0)
+    (effects (font (size 1.27 1.27)))
+  )
   (text "3V3"  (exclude_from_sim no)(at 252.73 94.742 0)
     (effects (font (size 1.27 1.27)))
@@
   (text "Barrel Jack"  (exclude_from_sim no)(at 147.32 102.108 0)
     (effects (font (size 1.27 1.27)))
+  )
+  (text "Non default font text"  (exclude_from_sim no)(at 41.656 245.364 0)
+    (effects (font (face "Lato") (size 2.54 2.54) (thickness 0.508) (bold yes)))
   )
   (text "Clock generator"  (exclude_from_sim no)(at 186.944 134.112 0)
@@
         )
       )
-    )
-  )
-  (symbol (lib_id "test_project:MountingHole_Pad") (at 368.3 236.22 270) (unit 1) (exclude_from_sim yes)
-    (in_bom no) (on_board yes) (dnp no) (fields_autoplaced yes)
-    (property "Reference" "H4" (at 372.11 234.9499 90)
-      (effects (font (size 1.27 1.27)) (justify left))
-    )
-    (property "Value" "MountingHole_Pad" (at 372.11 237.4899 90)
-      (effects (font (size 1.27 1.27)) (justify left))
-    )
-    (property "Footprint" "test_project-footprints:MountingHole_2.2mm_M2_DIN965_Pad" (at 368.3 236.22 0)
-      (effects (font (size 1.27 1.27))( hide yes ))
-    )
-    (property "Datasheet" "~" (at 368.3 236.22 0)
-      (effects (font (size 1.27 1.27))( hide yes ))
-    )
-    (property "Description" "Mounting Hole with connection" (at 368.3 236.22 0)
-      (effects (font (size 1.27 1.27))( hide yes ))
-    )
-  (pin  "1")
-    (instances
-      (project "test_project"
-        (path "/59f522e0-0cf7-48a6-bc09-47b340553d24"
-          (reference "H4") (unit 1)
-        )
-      )

Commit message: [#75441] Kicad9
Connections:
- no-connect marks 0 -> 1
Other:
- added sheet multi-channel-test (multi-channel-test.kicad_sch)
- added sheet multi-channel-test1 (multi-channel-test.kicad_sch)
