File: tests/test_project/receiver.kicad_sch (KiCad schematic)
At the start: 43 parts, among them U1 ASDMB-xxxMHz, U2 ADV7611

Commit message: [#70870] Update test design rebase
Changed lines of the file:
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@@
 	(label "P17"
 		(at 269.24 55.88 180)
-		(fields_autoplaced yes)
 		(effects
 			(font
@@
 	(label "ADV7611_CK_N"
 		(at 179.07 58.42 0)
-		(fields_autoplaced yes)
 		(effects
 			(font
@@
 	(label "hdmi_in.CEC"
 		(at 147.32 60.96 0)
-		(fields_autoplaced yes)
 		(effects
 			(font
@@
 	(label "P19"
 		(at 269.24 50.8 180)
-		(fields_autoplaced yes)
 		(effects
 			(font
@@
 	(label "ADV7611_D2_N"
 		(at 179.07 43.18 0)
-		(fields_autoplaced yes)
 		(effects
 			(font
@@
 	(label "P20"
 		(at 269.24 48.26 180)
-		(fields_autoplaced yes)
 		(effects
 			(font
@@
 	(label "P22"
 		(at 269.24 43.18 180)
-		(fields_autoplaced yes)
 		(effects
 			(font
@@
 	(label "P12"
 		(at 269.24 68.58 180)
-		(fields_autoplaced yes)
 		(effects
 			(font
@@
 	(label "ADV7611_D0_P"
 		(at 179.07 50.8 0)
-		(fields_autoplaced yes)
 		(effects
 			(font
@@
 	(label "hdmi_in.D0-"
 		(at 160.02 53.34 180)
-		(fields_autoplaced yes)
 		(effects
 			(font
@@
 	(label "P10"
 		(at 269.24 73.66 180)
-		(fields_autoplaced yes)
 		(effects
 			(font
@@
 	(label "hdmi_in.D1-"
 		(at 160.02 48.26 180)
-		(fields_autoplaced yes)
 		(effects
 			(font
@@
 	(label "xtal_p"
 		(at 182.88 123.19 180)
-		(fields_autoplaced yes)
 		(effects
 			(font
@@
 	(label "P23"
 		(at 269.24 40.64 180)
-		(fields_autoplaced yes)
 		(effects
 			(font
@@
 	(label "P0"
 		(at 269.24 99.06 180)
-		(fields_autoplaced yes)
 		(effects
 			(font
@@
 	(label "P16"
 		(at 269.24 58.42 180)
-		(fields_autoplaced yes)
 		(effects
 			(font
@@
 	(label "P5"
 		(at 269.24 86.36 180)
-		(fields_autoplaced yes)
 		(effects
 			(font
@@
 	(label "hdmi_in.D2-"
 		(at 160.02 43.18 180)
-		(fields_autoplaced yes)
 		(effects
 			(font
@@
 	(label "hdmi_in.SDA"
 		(at 158.75 66.04 180)
-		(fields_autoplaced yes)
 		(effects
 			(font
@@
 	(label "P21"
 		(at 269.24 45.72 180)
-		(fields_autoplaced yes)
 		(effects
 			(font
@@
 	(label "P4"
 		(at 269.24 88.9 180)
-		(fields_autoplaced yes)
 		(effects
 			(font
@@
 	(label "ADV7611_D1_P"
 		(at 179.07 45.72 0)
-		(fields_autoplaced yes)
 		(effects
 			(font
@@
 	(label "hdmi_in.CK+"
 		(at 160.02 55.88 180)
-		(fields_autoplaced yes)
 		(effects
 			(font
@@
 	(label "P14"
 		(at 269.24 63.5 180)
-		(fields_autoplaced yes)
 		(effects
 			(font
@@
 	(label "P15"
 		(at 269.24 60.96 180)
-		(fields_autoplaced yes)
 		(effects
 			(font
@@
 	(label "P13"
 		(at 269.24 66.04 180)
-		(fields_autoplaced yes)
 		(effects
 			(font
@@
 	(label "P9"
 		(at 269.24 76.2 180)
-		(fields_autoplaced yes)
 		(effects
 			(font
@@
 	(label "ADV7611_CK_P"
 		(at 179.07 55.88 0)
-		(fields_autoplaced yes)
 		(effects
 			(font
@@
 	(label "P18"
 		(at 269.24 53.34 180)
-		(fields_autoplaced yes)
 		(effects
 			(font
@@
 	(label "hdmi_in.D0+"
 		(at 160.02 50.8 180)
-		(fields_autoplaced yes)
 		(effects
 			(font
@@
 	(label "hdmi_in.D1+"
 		(at 160.02 45.72 180)
-		(fields_autoplaced yes)
 		(effects
 			(font
@@
 	(label "P1"
 		(at 269.24 96.52 180)
-		(fields_autoplaced yes)
 		(effects
 			(font
@@
 	(label "P7"
 		(at 269.24 81.28 180)
-		(fields_autoplaced yes)
 		(effects
 			(font
@@
 	(label "ADV7611_D0_N"
 		(at 179.07 53.34 0)
-		(fields_autoplaced yes)
 		(effects
 			(font
@@
 	(label "hdmi_in.D2+"
 		(at 160.02 40.64 180)
-		(fields_autoplaced yes)
 		(effects
 			(font
@@
 	(label "hdmi_in.CK-"
 		(at 160.02 58.42 180)
-		(fields_autoplaced yes)
 		(effects
 			(font
@@
 	(label "hdmi_in.SCL"
 		(at 158.75 63.5 180)
-		(fields_autoplaced yes)
 		(effects
 			(font
@@
 	(label "xtal_p"
 		(at 186.69 88.9 0)
-		(fields_autoplaced yes)
 		(effects
 			(font
@@
 	(label "ADV7611_D2_P"
 		(at 179.07 40.64 0)
-		(fields_autoplaced yes)
 		(effects
 			(font
@@
 	(label "ADV7611_D1_N"
 		(at 179.07 48.26 0)
-		(fields_autoplaced yes)
 		(effects
 			(font
@@
 	(label "P8"
 		(at 269.24 78.74 180)
-		(fields_autoplaced yes)
 		(effects
 			(font
@@
 	(label "P6"
 		(at 269.24 83.82 180)
-		(fields_autoplaced yes)
 		(effects
 			(font
@@
 	(label "P3"
 		(at 269.24 91.44 180)
-		(fields_autoplaced yes)
 		(effects
 			(font
@@
 	(label "P2"
 		(at 269.24 93.98 180)
-		(fields_autoplaced yes)
 		(effects
 			(font
@@
 	(label "P11"
 		(at 269.24 71.12 180)
-		(fields_autoplaced yes)
 		(effects
 			(font
@@
 	(label "hdmi_in.HPD"
 		(at 158.75 68.58 180)
-		(fields_autoplaced yes)
 		(effects
 			(font
@@
 		(shape input)
 		(at 144.78 38.1 180)
-		(fields_autoplaced yes)
 		(effects
 			(font
@@
 		(shape input)
 		(at 166.37 73.66 180)
-		(fields_autoplaced yes)
 		(effects
 			(font
@@
 		(shape input)
 		(at 267.97 119.38 0)
-		(fields_autoplaced yes)
 		(effects
 			(font
@@
 		(shape input)
 		(at 166.37 86.36 180)
-		(fields_autoplaced yes)
 		(effects
 			(font
@@
 		(shape input)
 		(at 267.97 106.68 0)
-		(fields_autoplaced yes)
 		(effects
 			(font
@@
 		(shape input)
 		(at 267.97 127 0)
-		(fields_autoplaced yes)
 		(effects
 			(font
@@
 		(shape input)
 		(at 267.97 111.76 0)
-		(fields_autoplaced yes)
 		(effects
 			(font
@@
 		(shape input)
 		(at 166.37 81.28 180)
-		(fields_autoplaced yes)
 		(effects
 			(font
@@
 		(shape input)
 		(at 267.97 104.14 0)
-		(fields_autoplaced yes)
 		(effects
 			(font
@@
 		(shape input)
 		(at 267.97 116.84 0)
-		(fields_autoplaced yes)
 		(effects
 			(font
@@
 		(shape input)
 		(at 271.78 38.1 0)
-		(fields_autoplaced yes)
 		(effects
 			(font
@@
 		(shape input)
 		(at 267.97 124.46 0)
-		(fields_autoplaced yes)
 		(effects
 			(font
@@
 		(shape input)
 		(at 267.97 109.22 0)
-		(fields_autoplaced yes)
 		(effects
 			(font
@@
 		)
 		(pin "51"
+			(alternate "INT2")
 		)
 		(pin "61"
