File: tests/test_project/test_project.kicad_sch (KiCad schematic)
At the start: 4 parts

Commit message: [#70870] Update test design rebase
Parts:
- removed H4: MountingHole_Pad, MountingHole:MountingHole_2.2mm_M2_DIN965_Pad, symbol Mechanical:MountingHole_Pad
Other:
- note added: "Arc > 180 deg"
- note added: "Non default font text"
- note added: "PNG image"
Changed lines of the file:
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@@
 		(color 0 0 0 0)
 	)
-	(junction
-		(at 365.76 236.22)
-		(diameter 0)
-		(color 0 0 0 0)
-	)
 	(polyline
 		(pts
@@
 	(polyline
 		(pts
-			(xy 251.1531 158.414) (xy 250.9414 135.5751)
+			(xy 250.9368 157.9439) (xy 250.9414 135.5751)
 		)
 		(stroke
@@
 	(wire
 		(pts
-			(xy 365.76 231.14) (xy 365.76 236.22)
-		)
-		(stroke
-			(width 0)
-			(type default)
-		)
-	)
-	(wire
-		(pts
-			(xy 365.76 236.22) (xy 365.76 240.03)
+			(xy 365.76 231.14) (xy 365.76 240.03)
 		)
 		(stroke
@@
 	(polyline
 		(pts
-			(xy 265.6258 134.0326) (xy 265.7237 158.2976)
+			(xy 265.6258 134.0326) (xy 265.6407 157.9838)
 		)
 		(stroke
@@
 		)
 		(fill
-			(type outline)
+			(type color)
+			(color 0 0 0 0)
 		)
 	)
@@
 		)
 		(fill
-			(type outline)
+			(type color)
+			(color 0 0 0 0)
 		)
 	)
@@
 		)
 		(fill
-			(type outline)
+			(type color)
+			(color 0 0 0 0)
 		)
 	)
@@
 		)
 		(fill
-			(type outline)
-		)
-	)
-	(polyline
-		(pts
-			(xy 251.1663 159.803) (xy 250.2217 157.9589) (xy 251.1531 158.414) (xy 252.0738 157.943) (xy 251.1663 159.803)
-		)
-		(stroke
-			(width 0)
-			(type solid)
-		)
-		(fill
-			(type outline)
+			(type color)
+			(color 0 0 0 0)
+		)
+	)
+	(arc
+		(start 49.53 219.71)
+		(mid 30.6664 215.265)
+		(end 49.53 210.82)
+		(stroke
+			(width 0)
+			(type default)
+		)
+		(fill
+			(type none)
+		)
+	)
+	(polyline
+		(pts
+			(xy 250.9966 159.6345) (xy 250.052 157.7904) (xy 250.9834 158.2455) (xy 251.9041 157.7745) (xy 250.9966 159.6345)
+		)
+		(stroke
+			(width 0)
+			(type solid)
+		)
+		(fill
+			(type color)
+			(color 0 0 0 0)
 		)
 	)
@@
 		)
 		(fill
-			(type outline)
+			(type color)
+			(color 0 0 0 0)
 		)
 	)
@@
 		)
 		(fill
-			(type outline)
+			(type color)
+			(color 0 0 0 0)
 		)
 	)
@@
 		)
 		(fill
-			(type outline)
+			(type color)
+			(color 0 0 0 0)
 		)
 	)
@@
 		)
 		(fill
-			(type outline)
-		)
-	)
-	(polyline
-		(pts
-			(xy 265.7316 159.6866) (xy 264.7976 157.8398) (xy 265.7237 158.2976) (xy 266.6497 157.8319) (xy 265.7316 159.6866)
-		)
-		(stroke
-			(width 0)
-			(type solid)
-		)
-		(fill
-			(type outline)
+			(type color)
+			(color 0 0 0 0)
+		)
+	)
+	(polyline
+		(pts
+			(xy 265.6633 159.6377) (xy 264.7293 157.7909) (xy 265.6554 158.2487) (xy 266.5814 157.783) (xy 265.6633 159.6377)
+		)
+		(stroke
+			(width 0)
+			(type solid)
+		)
+		(fill
+			(type color)
+			(color 0 0 0 0)
 		)
 	)
@@
 		)
 		(fill
-			(type outline)
+			(type color)
+			(color 0 0 0 0)
+		)
+	)
+	(image
+		(at 41.91 186.69)
+		(data "iVBORw0KGgoAAAANSUhEUgAAASwAAABkCAIAAACzY5qXAAABhWlDQ1BJQ0MgcHJvZmlsZQAAKJF9"
+			"kT1Iw0AcxV9TpVIrDmYQcchQnayDiggutQpFqBBqhVYdzEe/oElDkuLiKLgWHPxYrDq4OOvq4CoI"
+			"gh8gzg5Oii5S4v+SQosYD4778e7e4+4dwDUqimZ1xQFNt810MiFkc6tC6BW94BHGOGYlxTLmRDEF"
+			"3/F1jwBb72Isy//cn6NPzVsKEBCI44ph2sQbxNObtsF4n5hXSpJKfE48ZtIFiR+ZLnv8xrjoMscy"
+			"eTOTnifmiYViB8sdrJRMjXiKOKpqOuVzWY9VxluMtUpNad2TvTCS11eWmU5zGEksYgkiBMiooYwK"
+			"bMRo1UmxkKb9hI9/yPWL5JLJVYZCjgVUoUFy/WB/8LtbqzA54SVFEkD3i+N8jAChXaBZd5zvY8dp"
+			"ngDBZ+BKb/urDWDmk/R6W4seAf3bwMV1W5P3gMsdYPDJkEzJlYI0uUIBeD+jb8oBA7dAeM3rrbWP"
+			"0wcgQ12lboCDQ2C0SNnrPu/u6ezt3zOt/n4AClhy4x7yWMEAAAAJcEhZcwAALiMAAC4jAXilP3YA"
+			"AADwSURBVHja7dNBDQAgEAPBO6yBbNAGFvolmZHQdPsWkbNrTTPE2rNSwwQgQhAhIEIQISBCECEg"
+			"QhAhIEIQISBCECEgQhAhIEIQISBCECEgQhAhIEIQISBCECEgQhAhIEIQISBCECEgQhAhIEIQISBC"
+			"ECEgQhAhIEIQISBCECEgQhAhIEIQISBCECEgQhAhIEIQISBCECEgQhAhIEIQISBCECEgQhAhIEIQ"
+			"IYgQECGIEBAhiBAQIYgQECGIEBAhiBAQIYgQECGIEBAhiBAQIYgQECGIEBAhiBAQIYgQECGIEBAh"
+			"iBAQIYgQECGIEBAh/OwB8voExzrxYwwAAAAASUVORK5CYII="
 		)
 	)
@@
 		)
 	)
+	(text "Arc > 180 deg"
+		(exclude_from_sim no)
+		(at 40.894 215.646 0)
+		(effects
+			(font
+				(size 1.27 1.27)
+			)
+		)
+	)
+	(text "PNG image"
+		(exclude_from_sim no)
+		(at 41.91 180.848 0)
+		(effects
+			(font
+				(size 1.27 1.27)
+			)
+		)
+	)
 	(text "3V3"
 		(exclude_from_sim no)
@@
 			(font
 				(size 1.27 1.27)
+			)
+		)
+	)
+	(text "Non default font text"
+		(exclude_from_sim no)
+		(at 41.656 245.364 0)
+		(effects
+			(font
+				(face "Lato")
+				(size 2.54 2.54)
+				(thickness 0.508)
+				(bold yes)
 			)
 		)
@@
 					(unit 1)
 				)
-			)
-		)
-	)
-	(symbol
-		(lib_id "Mechanical:MountingHole_Pad")
-		(at 368.3 236.22 270)
-		(unit 1)
-		(exclude_from_sim yes)
-		(in_bom no)
-		(on_board yes)
-		(dnp no)
-		(fields_autoplaced yes)
-		(property "Reference" "H4"
-			(at 372.11 234.9499 90)
-			(effects
-				(font
-					(size 1.27 1.27)
-				)
-				(justify left)
-			)
-		)
-		(property "Value" "MountingHole_Pad"
-			(at 372.11 237.4899 90)
-			(effects
-				(font
-					(size 1.27 1.27)
-				)
-				(justify left)
-			)
-		)
-		(property "Footprint" "MountingHole:MountingHole_2.2mm_M2_DIN965_Pad"
-			(at 368.3 236.22 0)
-			(effects
-				(font
-					(size 1.27 1.27)
-				)
-				(hide yes)
-			)
-		)
-		(property "Datasheet" "~"
-			(at 368.3 236.22 0)
-			(effects
-				(font
-					(size 1.27 1.27)
-				)
-				(hide yes)
-			)
-		)
-		(property "Description" "Mounting Hole with connection"
-			(at 368.3 236.22 0)
-			(effects
-				(font
-					(size 1.27 1.27)
-				)
-				(hide yes)
-			)
-		)
-		(pin "1"
-		)
-		(instances
-			(project "test_project"
-				(path "/59f522e0-0cf7-48a6-bc09-47b340553d24"
-					(reference "H4")
-					(unit 1)
-				)

Commit message: [#75441] Kicad9
Connections:
- no-connect marks 0 -> 1
Other:
- added sheet multi-channel-test (multi-channel-test.kicad_sch)
- added sheet multi-channel-test1 (multi-channel-test.kicad_sch)
