File: tests/reference-outputs/kicad9/loclib/connectors.kicad_sch (KiCad schematic)
At the start: 6 parts, among them J1 HDMI_A, J2 Conn_01x02_Pin, J4 Conn_01x35_Pin

Commit message: [#93049] tests: Use askiff test project
Parts:
- C1: footprint Capacitor_SMD:C_0402_1005Metric -> test_project-footprints:C_0402_1005Metric; symbol Device:C -> test_project:C
- D3: footprint Package_TO_SOT_SMD:SOT-353_SC-70-5 -> test_project-footprints:SOT-353_SC-70-5; symbol Power_Protection:PESD3V3L4UG -> test_project:PESD3V3L4UG
- J1: footprint Connector_Video:HDMI_A_Amphenol_10029449-x01xLF_Horizontal -> test_project-footprints:HDMI_A_Amphenol_10029449-x01xLF_Horizontal; symbol Connector:HDMI_A -> test_project:HDMI_A
- J2: footprint Connector_JST:JST_XH_B2B-XH-AM_1x02_P2.50mm_Vertical -> test_project-footprints:JST_XH_B2B-XH-AM_1x02_P2.50mm_Vertical; symbol Connector:Conn_01x02_Pin -> test_project:Conn_01x02_Pin
- J4: footprint Connector_PinHeader_1.00mm:PinHeader_1x35_P1.00mm_Vertical_SMD_Pin1Left -> test_project-footprints:PinHeader_1x35_P1.00mm_Vertical_SMD_Pin1Left; symbol Connector:Conn_01x35_Pin -> test_project:Conn_01x35_Pin
- R11: footprint Resistor_SMD:R_0402_1005Metric -> test_project-footprints:R_0402_1005Metric; symbol Device:R -> test_project:R
Changed lines of the file:
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@@
 	)
 	(symbol
-		(lib_id "Connector:HDMI_A")
+		(lib_id "test_project:HDMI_A")
 		(at 90.17 105.41 0)
 		(unit 1)
@@
 			)
 		)
-		(property "Footprint" "Connector_Video:HDMI_A_Amphenol_10029449-x01xLF_Horizontal"
+		(property "Footprint" "test_project-footprints:HDMI_A_Amphenol_10029449-x01xLF_Horizontal"
 			(at 90.805 105.41 0)
 			(effects
@@
 	)
 	(symbol
-		(lib_id "power:PWR_FLAG")
+		(lib_id "test_project:PWR_FLAG")
 		(at 113.03 80.01 0)
 		(unit 1)
@@
 	)
 	(symbol
-		(lib_id "power:GND")
+		(lib_id "test_project:GND")
 		(at 97.79 137.16 0)
 		(mirror y)
@@
 	)
 	(symbol
-		(lib_id "Connector:Conn_01x02_Pin")
+		(lib_id "test_project:Conn_01x02_Pin")
 		(at 218.44 45.72 0)
 		(mirror y)
@@
 			)
 		)
-		(property "Footprint" "Connector_JST:JST_XH_B2B-XH-AM_1x02_P2.50mm_Vertical"
+		(property "Footprint" "test_project-footprints:JST_XH_B2B-XH-AM_1x02_P2.50mm_Vertical"
 			(at 218.44 45.72 0)
 			(effects
@@
 	)
 	(symbol
-		(lib_id "power:GND")
+		(lib_id "test_project:GND")
 		(at 55.88 137.16 0)
 		(mirror y)
@@
 	)
 	(symbol
-		(lib_id "Device:C")
+		(lib_id "test_project:C")
 		(at 105.41 73.66 0)
 		(mirror y)
@@
 			)
 		)
-		(property "Footprint" "Capacitor_SMD:C_0402_1005Metric"
+		(property "Footprint" "test_project-footprints:C_0402_1005Metric"
 			(at 104.4448 77.47 0)
 			(effects
@@
 	)
 	(symbol
-		(lib_id "power:GND")
+		(lib_id "test_project:GND")
 		(at 199.39 156.21 0)
 		(unit 1)
@@
 	)
 	(symbol
-		(lib_id "Power_Protection:PESD3V3L4UG")
+		(lib_id "test_project:PESD3V3L4UG")
 		(at 55.88 132.08 270)
 		(unit 1)
@@
 			)
 		)
-		(property "Footprint" "Package_TO_SOT_SMD:SOT-353_SC-70-5"
+		(property "Footprint" "test_project-footprints:SOT-353_SC-70-5"
 			(at 60.96 132.08 0)
 			(effects
@@
 	)
 	(symbol
-		(lib_id "power:+3V3")
+		(lib_id "test_project:+3V3")
 		(at 199.39 153.67 0)
 		(unit 1)
@@
 	)
 	(symbol
-		(lib_id "power:+5V")
+		(lib_id "test_project:+5V")
 		(at 27.94 109.22 0)
 		(unit 1)
@@
 	)
 	(symbol
-		(lib_id "Connector:Conn_01x35_Pin")
+		(lib_id "test_project:Conn_01x35_Pin")
 		(at 218.44 113.03 0)
 		(mirror y)
@@
 			)
 		)
-		(property "Footprint" "Connector_PinHeader_1.00mm:PinHeader_1x35_P1.00mm_Vertical_SMD_Pin1Left"
+		(property "Footprint" "test_project-footprints:PinHeader_1x35_P1.00mm_Vertical_SMD_Pin1Left"
 			(at 218.44 113.03 0)
 			(effects
@@
 	)
 	(symbol
-		(lib_id "Power_Protection:PESD3V3L4UG")
+		(lib_id "test_project:PESD3V3L4UG")
 		(at 60.96 132.08 270)
 		(unit 2)
@@
 			)
 		)
-		(property "Footprint" "Package_TO_SOT_SMD:SOT-353_SC-70-5"
+		(property "Footprint" "test_project-footprints:SOT-353_SC-70-5"
 			(at 66.04 132.08 0)
 			(effects
@@
 	)
 	(symbol
-		(lib_id "power:PWR_FLAG")
+		(lib_id "test_project:PWR_FLAG")
 		(at 105.41 67.31 0)
 		(unit 1)
@@
 	)
 	(symbol
-		(lib_id "Power_Protection:PESD3V3L4UG")
+		(lib_id "test_project:PESD3V3L4UG")
 		(at 71.12 132.08 270)
 		(unit 4)
@@
 			)
 		)
-		(property "Footprint" "Package_TO_SOT_SMD:SOT-353_SC-70-5"
+		(property "Footprint" "test_project-footprints:SOT-353_SC-70-5"
 			(at 76.2 132.08 0)
 			(effects
@@
 	)
 	(symbol
-		(lib_id "power:GND")
+		(lib_id "test_project:GND")
 		(at 105.41 81.28 0)
 		(mirror y)
@@
 	)
 	(symbol
-		(lib_id "power:+5V")
+		(lib_id "test_project:+5V")
 		(at 90.17 67.31 0)
 		(mirror y)
@@
 	)
 	(symbol
-		(lib_id "Power_Protection:PESD3V3L4UG")
+		(lib_id "test_project:PESD3V3L4UG")
 		(at 66.04 132.08 270)
 		(unit 3)
@@
 			)
 		)
-		(property "Footprint" "Package_TO_SOT_SMD:SOT-353_SC-70-5"
+		(property "Footprint" "test_project-footprints:SOT-353_SC-70-5"
 			(at 71.12 132.08 0)
 			(effects
@@
 	)
 	(symbol
-		(lib_id "Device:R")
+		(lib_id "test_project:R")
 		(at 27.94 114.3 0)
 		(unit 1)
@@
 			)
 		)
-		(property "Footprint" "Resistor_SMD:R_0402_1005Metric"
+		(property "Footprint" "test_project-footprints:R_0402_1005Metric"
 			(at 26.162 114.3 90)
 			(effects
