File: tests/reference-outputs/kicad9/loclib/multi-channel-test.kicad_sch (KiCad schematic)
At the start: 6 parts

Commit message: [#93049] tests: Use askiff test project
Parts:
- R13, R14, R15, R16: footprint Resistor_SMD:R_0402_1005Metric -> test_project-footprints:R_0402_1005Metric; symbol Device:R -> test_project:R
- TP5, TP6: footprint TestPoint:TestPoint_Pad_D1.0mm -> test_project-footprints:TestPoint_Pad_D1.0mm; symbol Connector:TestPoint -> test_project:TestPoint
Changed lines of the file:
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@@
 	)
 	(symbol
-		(lib_id "Device:R")
+		(lib_id "test_project:R")
 		(at 125.73 82.55 270)
 		(unit 1)
@@
 			)
 		)
-		(property "Footprint" "Resistor_SMD:R_0402_1005Metric"
+		(property "Footprint" "test_project-footprints:R_0402_1005Metric"
 			(at 125.73 80.772 90)
 			(effects
@@
 	)
 	(symbol
-		(lib_id "Device:R")
+		(lib_id "test_project:R")
 		(at 101.6 82.55 270)
 		(unit 1)
@@
 			)
 		)
-		(property "Footprint" "Resistor_SMD:R_0402_1005Metric"
+		(property "Footprint" "test_project-footprints:R_0402_1005Metric"
 			(at 101.6 80.772 90)
 			(effects
@@
 	)
 	(symbol
-		(lib_id "Device:R")
+		(lib_id "test_project:R")
 		(at 113.03 77.47 180)
 		(unit 1)
@@
 			)
 		)
-		(property "Footprint" "Resistor_SMD:R_0402_1005Metric"
+		(property "Footprint" "test_project-footprints:R_0402_1005Metric"
 			(at 114.808 77.47 90)
 			(effects
@@
 	)
 	(symbol
-		(lib_id "Connector:TestPoint")
+		(lib_id "test_project:TestPoint")
 		(at 133.35 82.55 270)
 		(unit 1)
@@
 			)
 		)
-		(property "Footprint" "TestPoint:TestPoint_Pad_D1.0mm"
+		(property "Footprint" "test_project-footprints:TestPoint_Pad_D1.0mm"
 			(at 133.35 87.63 0)
 			(effects
@@
 	)
 	(symbol
-		(lib_id "power:GND")
+		(lib_id "test_project:GND")
 		(at 113.03 93.98 0)
 		(unit 1)
@@
 	)
 	(symbol
-		(lib_id "Device:R")
+		(lib_id "test_project:R")
 		(at 113.03 88.9 180)
 		(unit 1)
@@
 			)
 		)
-		(property "Footprint" "Resistor_SMD:R_0402_1005Metric"
+		(property "Footprint" "test_project-footprints:R_0402_1005Metric"
 			(at 114.808 88.9 90)
 			(effects
@@
 	)
 	(symbol
-		(lib_id "Connector:TestPoint")
+		(lib_id "test_project:TestPoint")
 		(at 93.98 82.55 90)
 		(unit 1)
@@
 			)
 		)
-		(property "Footprint" "TestPoint:TestPoint_Pad_D1.0mm"
+		(property "Footprint" "test_project-footprints:TestPoint_Pad_D1.0mm"
 			(at 93.98 77.47 0)
 			(effects
@@
 	)
 	(symbol
-		(lib_id "power:+3V3")
+		(lib_id "test_project:+3V3")
 		(at 113.03 71.12 0)
 		(unit 1)
