File: tests/reference-outputs/kicad9/loclib/receiver.kicad_sch (KiCad schematic)
At the start: 43 parts, among them U1 ASDMB-xxxMHz, U2 ADV7611

Commit message: [#93049] tests: Use askiff test project
Parts:
- C10, C14, C15, C16, C17, C18, C19, C2, C20, C21, C22, C23, C24, C25, C26, C27, C28, C29, C3, C30, C31, C32, C33, C34, C35, C36, C37, C38, C39, C4, C5, C6, C7, C8, C9: footprint Capacitor_SMD:C_0402_1005Metric -> test_project-footprints:C_0402_1005Metric; symbol Device:C -> test_project:C
- R1, R10, R2, R3, R6, R7: footprint Resistor_SMD:R_0402_1005Metric -> test_project-footprints:R_0402_1005Metric; symbol Device:R -> test_project:R
- U1: footprint Oscillator:Oscillator_SMD_Abracon_ASDMB-4Pin_2.5x2.0mm -> test_project-footprints:Oscillator_SMD_Abracon_ASDMB-4Pin_2.5x2.0mm; symbol Oscillator:ASDMB-xxxMHz -> test_project:ASDMB-xxxMHz
- U2: footprint Package_QFP:LQFP-64-1EP_10x10mm_P0.5mm_EP5x5mm -> test_project-footprints:LQFP-64-1EP_10x10mm_P0.5mm_EP5x5mm; symbol Interface_HDMI:ADV7611 -> test_project:ADV7611
