File: tests/reference-outputs/kicad9/loclib/test_project.kicad_pcb (KiCad board)
At the start: 8 copper layers, 57.6 x 50 mm, 91 parts, among them J1 HDMI_A, J2 Conn_01x02_Pin, J3 Barrel_Jack_MountingPin, J4 Conn_01x35_Pin, U1 ASDMB-xxxMHz, U2 ADV7611, U3 LM3880, U4 AP2112K-1.8, U6 RT9742AGJ5F

Commit message: [#93049] tests: Use askiff test project
Parts:
- C1, C10, C11, C12, C13, C14, C15, C16, C17, C18, C19, C2, C20, C21, C22, C23, C24, C25, C26, C27, C28, C29, C3, C30, C31, C32, C33, C34, C35, C36, C37, C38, C39, C4, C40, C5, C6, C7, C8, C9, REF** (x4): footprint Capacitor_SMD:C_0402_1005Metric -> test_project-footprints:C_0402_1005Metric
- D1, D2: footprint LED_SMD:LED_0402_1005Metric -> test_project-footprints:LED_0402_1005Metric
- D3: footprint Package_TO_SOT_SMD:SOT-353_SC-70-5 -> test_project-footprints:SOT-353_SC-70-5
- FB1, FB2: footprint Inductor_SMD:L_0402_1005Metric -> test_project-footprints:L_0402_1005Metric
- H1, H2, H3: footprint MountingHole:MountingHole_2.2mm_M2_DIN965_Pad -> test_project-footprints:MountingHole_2.2mm_M2_DIN965_Pad
- J1: footprint Connector_Video:HDMI_A_Amphenol_10029449-x01xLF_Horizontal -> test_project-footprints:HDMI_A_Amphenol_10029449-x01xLF_Horizontal
- J2: footprint Connector_JST:JST_XH_B2B-XH-AM_1x02_P2.50mm_Vertical -> test_project-footprints:JST_XH_B2B-XH-AM_1x02_P2.50mm_Vertical
- J3: footprint Connector_BarrelJack:BarrelJack_CUI_PJ-063AH_Horizontal -> test_project-footprints:BarrelJack_CUI_PJ-063AH_Horizontal
- J4: footprint Connector_PinHeader_1.00mm:PinHeader_1x35_P1.00mm_Vertical_SMD_Pin1Left -> test_project-footprints:PinHeader_1x35_P1.00mm_Vertical_SMD_Pin1Left
- R1, R10, R11, R12, R13, R14, R15, R16, R17, R18, R19, R2, R20, R3, R4, R5, R6, R7, R8, R9: footprint Resistor_SMD:R_0402_1005Metric -> test_project-footprints:R_0402_1005Metric
- TP1, TP2, TP3, TP4, TP5, TP6, TP7, TP8: footprint TestPoint:TestPoint_Pad_D1.0mm -> test_project-footprints:TestPoint_Pad_D1.0mm
- U1: footprint Oscillator:Oscillator_SMD_Abracon_ASDMB-4Pin_2.5x2.0mm -> test_project-footprints:Oscillator_SMD_Abracon_ASDMB-4Pin_2.5x2.0mm
- U2: footprint Package_QFP:LQFP-64-1EP_10x10mm_P0.5mm_EP5x5mm -> test_project-footprints:LQFP-64-1EP_10x10mm_P0.5mm_EP5x5mm
- U3: footprint Package_TO_SOT_SMD:SOT-23-6 -> test_project-footprints:SOT-23-6
- U4, U6: footprint Package_TO_SOT_SMD:SOT-23-5 -> test_project-footprints:SOT-23-5
