File: tests/reference-outputs/kicad9/loclib/test_project.kicad_sch (KiCad schematic)
At the start: 3 parts

Commit message: [#93049] tests: Use askiff test project
Parts:
- H1, H2, H3: footprint MountingHole:MountingHole_2.2mm_M2_DIN965_Pad -> test_project-footprints:MountingHole_2.2mm_M2_DIN965_Pad; symbol Mechanical:MountingHole_Pad -> test_project:MountingHole_Pad
Changed lines of the file:
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@@
 	)
 	(symbol
-		(lib_id "Mechanical:MountingHole_Pad")
+		(lib_id "test_project:MountingHole_Pad")
 		(at 368.3 220.98 270)
 		(unit 1)
@@
 			)
 		)
-		(property "Footprint" "MountingHole:MountingHole_2.2mm_M2_DIN965_Pad"
+		(property "Footprint" "test_project-footprints:MountingHole_2.2mm_M2_DIN965_Pad"
 			(at 368.3 220.98 0)
 			(effects
@@
 	)
 	(symbol
-		(lib_id "Mechanical:MountingHole_Pad")
+		(lib_id "test_project:MountingHole_Pad")
 		(at 368.3 226.06 270)
 		(unit 1)
@@
 			)
 		)
-		(property "Footprint" "MountingHole:MountingHole_2.2mm_M2_DIN965_Pad"
+		(property "Footprint" "test_project-footprints:MountingHole_2.2mm_M2_DIN965_Pad"
 			(at 368.3 226.06 0)
 			(effects
@@
 	)
 	(symbol
-		(lib_id "Mechanical:MountingHole_Pad")
+		(lib_id "test_project:MountingHole_Pad")
 		(at 368.3 231.14 270)
 		(unit 1)
@@
 			)
 		)
-		(property "Footprint" "MountingHole:MountingHole_2.2mm_M2_DIN965_Pad"
+		(property "Footprint" "test_project-footprints:MountingHole_2.2mm_M2_DIN965_Pad"
 			(at 368.3 231.14 0)
 			(effects
@@
 	)
 	(symbol
-		(lib_id "Graphic:Logo_Open_Hardware_Large")
+		(lib_id "test_project:Logo_Open_Hardware_Large")
 		(at 39.37 266.7 0)
 		(unit 1)
@@
 	)
 	(symbol
-		(lib_id "power:GND")
+		(lib_id "test_project:GND")
 		(at 365.76 240.03 0)
 		(unit 1)
